File: kicad/printplaat.kicad_pcb (KiCad board)
At the start: 2 copper layers, 55.9 x 55.9 mm, 9 parts, among them J1 USB_B, U1 DFPlayerMini, U2 ATtiny85-20PU

Commit message: pcb and firmware v3
Parts:
- removed C1: 47nF, Capacitor_THT:C_Disc_D3.4mm_W2.1mm_P2.50mm
- added CP2: 1uF, Capacitor_THT:CP_Radial_D5.0mm_P2.50mm, F.Cu at (144.4, 135.6)
- added D1: LED, LED_THT:LED_D5.0mm, F.Cu at (100.3, 140.8)
- added J2: AVR-ISP-6, Connector_PinHeader_2.54mm:PinHeader_2x03_P2.54mm_Vertical, F.Cu at (144.0, 161.0)
- added JP1: SolderJumper_2_Open, Jumper:SolderJumper-2_P1.3mm_Open_RoundedPad1.0x1.5mm, F.Cu at (144.3, 149.8)
- added JP2: SolderJumper_2_Open, Jumper:SolderJumper-2_P1.3mm_Open_RoundedPad1.0x1.5mm, F.Cu at (146.8, 149.9)
- added R2: 220R, Resistor_THT:R_Axial_DIN0207_L6.3mm_D2.5mm_P10.16mm_Horizontal, F.Cu at (109.2, 128.3)
- R3: value 220R -> 10K
- R4: value 330K -> 220
- moved R3 44.2 mm to (99.7, 118.1), turned to 270 degrees
- moved R4 8.52 mm to (106.0, 118.1)
- moved R1 4.02 mm to (102.9, 118.1)
- moved CP1 3.47 mm to (144.4, 141.5), turned to 0 degrees
- moved U1 1.65 mm to (122.3, 124.5)
Connections:
- J1 pad 5: Net-(J1-Pad5) -> GND
- R1 pad 2: TX -> SCK
- R3 pad 1: Net-(R3-Pad1) -> PHONE
- R3 pad 2: PHONE -> Net-(CP2-Pad1)
- R4 pad 1: PHONE -> GND
- R4 pad 2: Net-(C1-Pad1) -> Net-(D1-Pad1)
- U1 pad 14: USB+ -> Net-(JP2-Pad1)
- U1 pad 15: USB- -> Net-(JP1-Pad1)
- U1 pad 3: RX -> MISO
- U1 pad 8: Net-(R3-Pad1) -> Net-(R2-Pad1)
- U2 pad 1: Net-(U2-Pad1) -> RST
- U2 pad 2: TX -> Net-(CP2-Pad1)
- U2 pad 3: RX -> BUSY
- U2 pad 5: Net-(U2-Pad5) -> MOSI
- U2 pad 6: BUSY -> MISO
- U2 pad 7: Net-(C1-Pad1) -> SCK
Routing:
- net MISO: track 0.00 -> 102.6 mm
- net Net-(CP2-Pad1): track 0.00 -> 93.6 mm
- net SCK: track 0.00 -> 81.3 mm
- net USB-: track 111.8 -> 35.9 mm, vias 1 -> 0
- net MOSI: track 0.00 -> 73.4 mm
- net USB+: track 102.1 -> 36.0 mm, vias 1 -> 0
- net Net-(JP1-Pad1): track 0.00 -> 58.8 mm
- net Net-(JP2-Pad1): track 0.00 -> 56.7 mm
- net RST: track 0.00 -> 49.2 mm
- net RX: track 48.4 -> 0.00 mm
- net Net-(C1-Pad1): track 33.9 -> 0.00 mm
- net TX: track 32.1 -> 0.00 mm
- net Net-(R2-Pad1): track 0.00 -> 24.1 mm
- net Net-(D1-Pad1): track 0.00 -> 18.8 mm
- net Net-(R3-Pad1): track 12.6 -> 0.00 mm
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Other:
- board text added: "1"
- board text added: "CUTOUT"
- board text added: "ICSP"
- board text added: "USB"
- board text added: "Wonderfoon mini V3"
