File: kicad/printplaat.sch (KiCad schematic (older format))
At the start: 9 parts, among them J1 USB_B, U1 DFPlayerMini, U2 ATtiny85-20PU

Commit message: pcb and firmware v3
Parts:
- removed C1: 47nF, Capacitor_THT:C_Disc_D3.4mm_W2.1mm_P2.50mm, symbol Device:C
- added CP2: 1uF, Capacitor_THT:CP_Radial_D5.0mm_P2.50mm, symbol Device:CP
- added D1: LED, LED_THT:LED_D5.0mm, symbol Device:LED
- added J2: AVR-ISP-6, Connector_PinHeader_2.54mm:PinHeader_2x03_P2.54mm_Vertical, symbol Connector:AVR-ISP-6
- added JP1, JP2: SolderJumper_2_Open, Jumper:SolderJumper-2_P1.3mm_Open_RoundedPad1.0x1.5mm, symbol Jumper:SolderJumper_2_Open
- added R4: 220, Resistor_THT:R_Axial_DIN0207_L6.3mm_D2.5mm_P10.16mm_Horizontal, symbol Device:R
- R3: renamed from R4; value 330K -> 10K
- renumbered R3 to R2
Connections:
- net BUSY: now also U2.3 (XTAL2/PB4); no longer U2.6 (PB1)
- net GND: now also J1.5 (Shield), CP2.2, J2.6 (GND), R4.1
- net USB+: now also JP2.2 (B); no longer U1.14 (USB+)
- net USB-: now also JP1.2 (B); no longer U1.15 (USB-)
- net VCC: now also J2.2 (VCC)
- net at R3.2: now also U2.2 (XTAL1/PB3), CP2.1; no longer U2.7 (PB2)
- net RST: now reaches U2.1 (~RESET~/PB5)
- net RST: now also J2.5 (~RST)
- net MOSI: now reaches U2.5 (AREF/PB0)
- net MOSI: now also D1.2 (A), J2.4 (MOSI)
- net RX renamed MISO
- net MISO: now also U2.6 (PB1), J2.1 (MISO); no longer U2.3 (XTAL2/PB4)
- net TX renamed SCK
- net SCK: now also U2.7 (PB2), J2.3 (SCK); no longer U2.2 (XTAL1/PB3)
- new net: JP2.1 (A), U1.14 (USB+)
- new net: JP1.1 (A), U1.15 (USB-)
- new net: D1.1 (K), R4.2
- no-connect marks 10 -> 7
Other:
- moved on the sheet: R3, U2
